File: hardware/kicad/pneuma-main/pneuma-main.kicad_pcb (KiCad board)
At the start: 4 copper layers, 43.2 x 45.1 mm, 63 parts, among them J1 TC2030-NL, J2 SPK, J3 LRA, J4 CAMERA, J5 TO_PWR, U1 Core11061408, U2 TPS22917DBVR, U3 MDBT50Q-1MV2, U4 MAX98357AETE+T, U5 DRV2605LDGSR, Y1 32.768k

Commit message: Move the touch pad under the camera bump, per the intended interaction
The touch area was over the battery, following K's "thin touch area" on the
lower front face.  It should sit ~10 mm below the camera bump, where a finger
lands: a 24 x 16 mm electrode at x -12..12, y -12..4 on the front membrane.

Consequences carried through:
- the AT42QT1011 front-end moves from PNM-PWR to PNM-MAIN beside the nRF, so
  the electrode run is short and TOUCH_OUT no longer crosses the FFC.  FFC pin
  27 becomes GND
- the electrode contacts PNM-MAIN TP11 at (11.0, 4.6)
- the speaker moves +2.2 mm in y to clear the pad.  It stays the 1 W 15 mm
  round part: the only sub-15 mm options are 5 mW earpiece receivers, and the
  15x11 alternative is 0.3 W (~5 dB quieter)
- the copper spreader keep-out follows the pad

Sensitivity is now the open question: the battery pouch is 1-2 mm behind the
pad's lower half and the speaker sits just above it.  Both are in REV-A.md as
bench-tuning items (Cs, and a foam spacer to hold the electrode off the metal).
Parts:
- added C24: 100n, C_0402_1005Metric, B.Cu at (109.8, 63.0)
- added C25: 22n, C_0402_1005Metric, B.Cu at (103.8, 95.5)
- added R15: 4.7k, R_0402_1005Metric, B.Cu at (100.3, 88.5)
- added TP11: TOUCH_E, SpringPad_3.0x2.0mm, F.Cu at (111.0, 95.4)
- added U6: AT42QT1011-MAH, DFN-8-1EP_2x2mm_P0.5mm_EP0.9x1.5mm, B.Cu at (114.3, 84.5)
- moved R10 12.3 mm to (103.3, 90.0)
- moved C13 12.2 mm to (103.8, 92.0), turned to 90 degrees
- moved R14 6.02 mm to (115.8, 63.5)
- moved R3 3.61 mm to (113.8, 66.5), turned to 0 degrees
- moved C14 3.54 mm to (113.8, 82.5)
Connections:
- J5 pad 27: TOUCH_OUT -> GND
