File: hardware/kicad/pneuma-pwr/interconnect.kicad_sch (KiCad schematic)
At the start: 6 parts, among them J5 TO_MAIN, U9 AT42QT1011-MAH

Commit message: Move the touch pad under the camera bump, per the intended interaction
The touch area was over the battery, following K's "thin touch area" on the
lower front face.  It should sit ~10 mm below the camera bump, where a finger
lands: a 24 x 16 mm electrode at x -12..12, y -12..4 on the front membrane.

Consequences carried through:
- the AT42QT1011 front-end moves from PNM-PWR to PNM-MAIN beside the nRF, so
  the electrode run is short and TOUCH_OUT no longer crosses the FFC.  FFC pin
  27 becomes GND
- the electrode contacts PNM-MAIN TP11 at (11.0, 4.6)
- the speaker moves +2.2 mm in y to clear the pad.  It stays the 1 W 15 mm
  round part: the only sub-15 mm options are 5 mW earpiece receivers, and the
  15x11 alternative is 0.3 W (~5 dB quieter)
- the copper spreader keep-out follows the pad

Sensitivity is now the open question: the battery pouch is 1-2 mm behind the
pad's lower half and the speaker sits just above it.  Both are in REV-A.md as
bench-tuning items (Cs, and a foam spacer to hold the electrode off the metal).
Parts:
- removed C22: 100n, Capacitor_SMD:C_0402_1005Metric, symbol Device:C
- removed C23: 22n, Capacitor_SMD:C_0402_1005Metric, symbol Device:C
- removed R20: 4.7k, Resistor_SMD:R_0402_1005Metric, symbol Device:R
- removed TP13: TOUCH_E, Pneuma:SpringPad_3.0x2.0mm, symbol Connector:TestPoint
- removed U9: AT42QT1011-MAH, Package_DFN_QFN:DFN-8-1EP_2x2mm_P0.5mm_EP0.9x1.5mm, symbol Sensor_Touch:AT42QT1011-M
Connections:
- net TOUCH_OUT is gone; now on net GND: J5.27 (Pin_27)
